Commit message: Add base_footprint for TF tree

File: urdf/robot.urdf (robot description, URDF)
Before this commit: robot diff_drive_robot, 4 links, 3 joints
Links:
- added link base_footprint
Joints:
- added joint base_footprint_to_base_link: type fixed, parent base_footprint, child base_link, origin xyz=0.0 0.0 0.0323 rpy=0 0 0
- joint lidar_joint: origin xyz=0.0 0.0 0.25 rpy=0 0 -1.5708 -> xyz=0.0 0.0 0.240 rpy=0 0 -1.5708
